File: HC2000_3.kicad_sch (KiCad schematic)
At the start: 9 parts

Commit message: Fix errors (IC & unnoticed cut for 1 EPROM)
Parts:
- UC3: value 7432N -> 74LS32
- UD4: value 74157N -> 74LS157
- UG4: value 7404N -> 74LS04
- UH3: value 7400N -> 74LS00
Changed lines of the file:
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@@
       (effects (font (size 1.778 1.5113)) (justify left bottom))
     )
-    (property "Value" "7404N" (at 220.98 38.1 0)
+    (property "Value" "74LS04" (at 220.98 38.1 0)
       (effects (font (size 1.778 1.5113)) (justify left bottom))
     )
@@
       (effects (font (size 1.778 1.5113)) (justify left bottom))
     )
-    (property "Value" "7404N" (at 220.98 68.58 0)
+    (property "Value" "74LS04" (at 220.98 68.58 0)
       (effects (font (size 1.778 1.5113)) (justify left bottom))
     )
@@
       (effects (font (size 1.778 1.5113)) (justify left bottom))
     )
-    (property "Value" "74157N" (at 208.28 134.62 0)
+    (property "Value" "74LS157" (at 208.28 134.62 0)
       (effects (font (size 1.778 1.5113)) (justify left bottom))
     )
@@
       (effects (font (size 1.778 1.5113)) (justify left bottom))
     )
-    (property "Value" "7432N" (at 208.28 152.4 0)
+    (property "Value" "74LS32" (at 208.28 152.4 0)
       (effects (font (size 1.778 1.5113)) (justify left bottom))
     )
@@
       (effects (font (size 1.778 1.5113)) (justify left bottom))
     )
-    (property "Value" "7404N" (at 220.98 53.34 0)
+    (property "Value" "74LS04" (at 220.98 53.34 0)
       (effects (font (size 1.778 1.5113)) (justify left bottom))
     )
@@
       (effects (font (size 1.778 1.5113)) (justify left bottom))
     )
-    (property "Value" "7400N" (at 68.58 45.72 0)
+    (property "Value" "74LS00" (at 68.58 45.72 0)
       (effects (font (size 1.778 1.5113)) (justify left bottom))
     )
@@
       (effects (font (size 1.778 1.5113)) (justify left bottom))
     )
-    (property "Value" "7404N" (at 73.66 132.08 0)
-      (effects (font (size 1.778 1.5113)) (justify left bottom))
-    )
+    (property "Value" "74LS04" (at 73.66 132.08 0)
+      (effects (font (size 1.778 1.5113)) (justify left bottom))
+    )
