File: HC2000_10.kicad_sch (KiCad schematic)
At the start: 16 parts

Commit message: Fix errors (IC & unnoticed cut for 1 EPROM)
Parts:
- UA11: value 7406N -> 74LS06
- UB9: value 74174N -> 74LS174
- UC10: value 74LS38N -> 74LS38
- UC9: value 74125N -> 74LS125
- UD11: value 7414N -> 74LS14
- UE11: value 7404N -> 74LS04
- UF8: value 74138N -> 74LS138
- UF9, UG9, UH8: value 7432N -> 74LS32
Changed lines of the file:
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@@
       (effects (font (size 1.778 1.5113)) (justify left bottom))
     )
-    (property "Value" "74LS38N" (at 160.02 83.82 0)
+    (property "Value" "74LS38" (at 160.02 83.82 0)
       (effects (font (size 1.778 1.5113)) (justify left bottom))
     )
@@
       (effects (font (size 1.778 1.5113)) (justify left bottom))
     )
-    (property "Value" "7432N" (at 99.06 182.88 0)
+    (property "Value" "74LS32" (at 99.06 182.88 0)
       (effects (font (size 1.778 1.5113)) (justify left bottom))
     )
@@
       (effects (font (size 1.778 1.5113)) (justify left bottom))
     )
-    (property "Value" "7432N" (at 99.06 104.14 0)
+    (property "Value" "74LS32" (at 99.06 104.14 0)
       (effects (font (size 1.778 1.5113)) (justify left bottom))
     )
@@
       (effects (font (size 1.778 1.5113)) (justify left bottom))
     )
-    (property "Value" "7432N" (at 99.06 139.7 0)
+    (property "Value" "74LS32" (at 99.06 139.7 0)
       (effects (font (size 1.778 1.5113)) (justify left bottom))
     )
@@
       (effects (font (size 1.778 1.5113)) (justify left bottom))
     )
-    (property "Value" "7432N" (at 99.06 121.92 0)
+    (property "Value" "74LS32" (at 99.06 121.92 0)
       (effects (font (size 1.778 1.5113)) (justify left bottom))
     )
@@
       (effects (font (size 1.778 1.5113)) (justify left bottom))
     )
-    (property "Value" "7432N" (at 60.96 121.92 0)
+    (property "Value" "74LS32" (at 60.96 121.92 0)
       (effects (font (size 1.778 1.5113)) (justify left bottom))
     )
@@
       (effects (font (size 1.778 1.5113)) (justify left bottom))
     )
-    (property "Value" "74LS38N" (at 160.02 101.6 0)
+    (property "Value" "74LS38" (at 160.02 101.6 0)
       (effects (font (size 1.778 1.5113)) (justify left bottom))
     )
@@
       (effects (font (size 1.778 1.5113)) (justify left bottom))
     )
-    (property "Value" "7432N" (at 60.96 86.36 0)
+    (property "Value" "74LS32" (at 60.96 86.36 0)
       (effects (font (size 1.778 1.5113)) (justify left bottom))
     )
@@
       (effects (font (size 1.778 1.5113)) (justify left bottom))
     )
-    (property "Value" "74LS38N" (at 160.02 48.26 0)
+    (property "Value" "74LS38" (at 160.02 48.26 0)
       (effects (font (size 1.778 1.5113)) (justify left bottom))
     )
@@
       (effects (font (size 1.778 1.5113)) (justify left bottom))
     )
-    (property "Value" "74LS38N" (at 160.02 66.04 0)
+    (property "Value" "74LS38" (at 160.02 66.04 0)
       (effects (font (size 1.778 1.5113)) (justify left bottom))
     )
@@
       (effects (font (size 1.778 1.5113)) (justify left bottom))
     )
-    (property "Value" "7414N" (at 219.71 45.72 0)
+    (property "Value" "74LS14" (at 219.71 45.72 0)
       (effects (font (size 1.778 1.778)) (justify left bottom))
     )
@@
       (effects (font (size 1.778 1.5113)) (justify left bottom))
     )
-    (property "Value" "7432N" (at 99.06 165.1 0)
+    (property "Value" "74LS32" (at 99.06 165.1 0)
       (effects (font (size 1.778 1.5113)) (justify left bottom))
     )
@@
       (effects (font (size 1.778 1.5113)) (justify left bottom))
     )
-    (property "Value" "74125N" (at 144.78 162.56 0)
+    (property "Value" "74LS125" (at 144.78 162.56 0)
       (effects (font (size 1.778 1.5113)) (justify left bottom))
     )
@@
       (effects (font (size 1.778 1.5113)) (justify left bottom))
     )
-    (property "Value" "7404N" (at 170.18 162.56 0)
+    (property "Value" "74LS04" (at 170.18 162.56 0)
       (effects (font (size 1.778 1.5113)) (justify left bottom))
     )
@@
       (effects (font (size 1.778 1.5113)) (justify left bottom))
     )
-    (property "Value" "74138N" (at 58.42 182.88 0)
+    (property "Value" "74LS138" (at 58.42 182.88 0)
       (effects (font (size 1.778 1.5113)) (justify left bottom))
     )
@@
       (effects (font (size 1.778 1.5113)) (justify left bottom))
     )
-    (property "Value" "7406N" (at 109.22 58.42 0)
+    (property "Value" "74LS06" (at 109.22 58.42 0)
       (effects (font (size 1.778 1.5113)) (justify left bottom) hide)
     )
@@
       (effects (font (size 1.778 1.5113)) (justify left bottom))
     )
-    (property "Value" "7432N" (at 60.96 139.7 0)
+    (property "Value" "74LS32" (at 60.96 139.7 0)
       (effects (font (size 1.778 1.5113)) (justify left bottom))
     )
@@
       (effects (font (size 1.778 1.5113)) (justify left bottom))
     )
-    (property "Value" "7432N" (at 60.96 104.14 0)
+    (property "Value" "74LS32" (at 60.96 104.14 0)
       (effects (font (size 1.778 1.5113)) (justify left bottom))
     )
@@
       (effects (font (size 1.778 1.5113)) (justify left bottom))
     )
-    (property "Value" "74174N" (at 60.96 60.96 0)
+    (property "Value" "74LS174" (at 60.96 60.96 0)
       (effects (font (size 1.778 1.5113)) (justify left bottom))
     )
@@
       (effects (font (size 1.778 1.5113)) (justify left bottom))
     )
-    (property "Value" "7432N" (at 99.06 86.36 0)
-      (effects (font (size 1.778 1.5113)) (justify left bottom))
-    )
+    (property "Value" "74LS32" (at 99.06 86.36 0)
+      (effects (font (size 1.778 1.5113)) (justify left bottom))
+    )

Commit message: Revision-E
Parts:
- C4: value 3,3uF/4,7uF -> 4,7uF
- R21: value 10k/470k -> 470k
Changed lines of the file:
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@@
       (effects (font (size 1.778 1.5113)) (justify left bottom))
     )
-    (property "Value" "10k/470k" (at 150.622 125.73 0)
+    (property "Value" "470k" (at 150.622 125.73 0)
       (effects (font (size 1.778 1.5113)) (justify left bottom))
     )
@@
       (effects (font (size 1.778 1.5113)) (justify left bottom))
     )
-    (property "Value" "3,3uF/4,7uF" (at 136.017 119.8626 0)
+    (property "Value" "4,7uF" (at 136.017 119.8626 0)
       (effects (font (size 1.778 1.5113)) (justify left bottom))
     )
