File: HC2000_15.kicad_sch (KiCad schematic)
At the start: 72 parts

Commit message: Updated ICs values and positions
Parts:
- UA8: value 2k x 4bit -> 2k x 4bit/-
- UB6: value ROM - 27C256 -> 27C256/27C512
Changed lines of the file:
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@@
       (effects (font (size 1.778 1.5113)) (justify left bottom))
     )
-    (property "Value" "ROM - 27C256" (at 46.99 116.84 0)
+    (property "Value" "27C256/27C512" (at 46.99 116.84 0)
       (effects (font (size 1.778 1.5113)) (justify left bottom) hide)
     )
@@
       (effects (font (size 1.778 1.5113)) (justify left bottom))
     )
-    (property "Value" "2k x 4bit" (at 53.34 81.28 0)
+    (property "Value" "2k x 4bit/-" (at 53.34 81.28 0)
       (effects (font (size 1.778 1.5113)) (justify left bottom) hide)
     )
@@
       (effects (font (size 1.778 1.5113)) (justify left bottom))
     )
-    (property "Value" "2k x 4bit" (at 80.01 137.16 0)
-      (effects (font (size 1.778 1.5113)) (justify left bottom) hide)
-    )
+    (property "Value" "2k x 4bit/-" (at 80.01 137.16 0)
+      (effects (font (size 1.778 1.5113)) (justify left bottom) hide)
+    )

Commit message: Fix errors (IC & unnoticed cut for 1 EPROM)
Parts:
- UA1, UC7: value 74244N -> 74LS244
- UA11: value 7406N -> 74LS06
- UA23, UA34: value 7409N -> 74LS09
- UA8: value 2k x 4bit/- -> 2k x 4bit CMOS RAM/-
- UA9, UB10, UE4, UF8, UH10: value 74138N -> 74LS138
- UB1, UD10, UD3, UE10, UF10, UF4, UG12, UH12: value 7474N -> 74LS74
- UB12: value 74153N -> 74LS153
- UB2, UH3: value 7400N -> 74LS00
- UB3: value 74367N -> 74LS367
- UB9, UF7: value 74174N -> 74LS174
- UC1, UE11, UG0, UG4: value 7404N -> 74LS04
- UC10: value 74LS38N -> 74LS38
- UC12, UF3, UG3, UH1: value 74175N -> 74LS175
- UC2: value 7427N -> 74LS27
- UC3, UE3, UF9, UG9, UH8: value 7432N -> 74LS32
- UC4, UC5, UD5, UG7, UH6: value 74257N -> 74LS257
- UC6: value 74373N -> 74LS373
- UC9: value 74125N -> 74LS125
- UD1, UE2, UG11: value 7408N -> 74LS08
- UD11: value 7414N -> 74LS14
- UD12: value 74LS161N -> 74LS161
- UD4: value 74157N -> 74LS157
- UD6, UF6, UG6: value 74374N -> 74LS374
- UE6: value 74166N -> 74LS166
- UG1: value 7442N -> 74LS42
- UG10, UH5: value 7400N -> 74LS08; symbol HC2000:7400N -> HC2000:7408N
- UG8: value 7405N -> 74LS05
- UH11: value 7493N -> 74LS93
- UH4: value 7486N -> 74LS86

Commit message: Revision-E
Parts:
- UA8: value 2k x 4bit CMOS RAM/- -> -
- UB6: value 27C256/27C512 -> 27C512
Changed lines of the file:
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@@
       (effects (font (size 1.778 1.5113)) (justify left bottom))
     )
-    (property "Value" "27C256/27C512" (at 46.99 116.84 0)
+    (property "Value" "27C512" (at 46.99 116.84 0)
       (effects (font (size 1.778 1.5113)) (justify left bottom) hide)
     )
@@
       (effects (font (size 1.778 1.5113)) (justify left bottom))
     )
-    (property "Value" "2k x 4bit CMOS RAM/-" (at 53.34 81.28 0)
+    (property "Value" "-" (at 53.34 81.28 0)
       (effects (font (size 1.778 1.5113)) (justify left bottom) hide)
     )
@@
       (effects (font (size 1.778 1.5113)) (justify left bottom))
     )
-    (property "Value" "2k x 4bit CMOS RAM/-" (at 80.01 137.16 0)
-      (effects (font (size 1.778 1.5113)) (justify left bottom) hide)
-    )
+    (property "Value" "-" (at 80.01 137.16 0)
+      (effects (font (size 1.778 1.5113)) (justify left bottom) hide)
+    )
