File: HC2000_7.kicad_sch (KiCad schematic)
At the start: 20 parts

Commit message: Fix errors (IC & unnoticed cut for 1 EPROM)
Parts:
- UD6, UF6, UG6: value 74374N -> 74LS374
- UE6: value 74166N -> 74LS166
- UH1: value 74175N -> 74LS175
- UH3: value 7400N -> 74LS00
- UH4: value 7486N -> 74LS86
- UH6: value 74257N -> 74LS257
Changed lines of the file:
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@@
       (effects (font (size 1.778 1.5113)) (justify left bottom))
     )
-    (property "Value" "74175N" (at 198.12 78.74 0)
+    (property "Value" "74LS175" (at 198.12 78.74 0)
       (effects (font (size 1.778 1.5113)) (justify left bottom))
     )
@@
       (effects (font (size 1.778 1.5113)) (justify left bottom))
     )
-    (property "Value" "74374N" (at 198.12 162.56 0)
+    (property "Value" "74LS374" (at 198.12 162.56 0)
       (effects (font (size 1.778 1.5113)) (justify left bottom))
     )
@@
       (effects (font (size 1.778 1.5113)) (justify left bottom))
     )
-    (property "Value" "74257N" (at 142.24 78.74 0)
+    (property "Value" "74LS257" (at 142.24 78.74 0)
       (effects (font (size 1.778 1.5113)) (justify left bottom))
     )
@@
       (effects (font (size 1.778 1.5113)) (justify left bottom))
     )
-    (property "Value" "74374N" (at 86.36 162.56 0)
+    (property "Value" "74LS374" (at 86.36 162.56 0)
       (effects (font (size 1.778 1.5113)) (justify left bottom))
     )
@@
       (effects (font (size 1.778 1.5113)) (justify left bottom))
     )
-    (property "Value" "7486N" (at 152.4 86.36 0)
+    (property "Value" "74LS86" (at 152.4 86.36 0)
       (effects (font (size 1.778 1.5113)) (justify left bottom))
     )
@@
       (effects (font (size 1.778 1.5113)) (justify left bottom))
     )
-    (property "Value" "7400N" (at 152.4 121.92 0)
+    (property "Value" "74LS00" (at 152.4 121.92 0)
       (effects (font (size 1.778 1.5113)) (justify left bottom))
     )
@@
       (effects (font (size 1.778 1.5113)) (justify left bottom))
     )
-    (property "Value" "74166N" (at 86.36 124.46 0)
+    (property "Value" "74LS166" (at 86.36 124.46 0)
       (effects (font (size 1.778 1.5113)) (justify left bottom))
     )
@@
       (effects (font (size 1.778 1.5113)) (justify left bottom))
     )
-    (property "Value" "74374N" (at 86.36 78.74 0)
-      (effects (font (size 1.778 1.5113)) (justify left bottom))
-    )
+    (property "Value" "74LS374" (at 86.36 78.74 0)
+      (effects (font (size 1.778 1.5113)) (justify left bottom))
+    )

Commit message: Revision-E
Parts:
- R6: value 2M2/2M -> 2M
Changed lines of the file:
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@@
       (effects (font (size 1.778 1.5113)) (justify left bottom))
     )
-    (property "Value" "2M2/2M" (at 156.21 153.162 0)
+    (property "Value" "2M" (at 156.21 153.162 0)
       (effects (font (size 1.778 1.5113)) (justify left bottom))
     )
