File: HC2000.kicad_pcb (KiCad board)
At the start: 2 copper layers, 478 x 183 mm, 255 parts, among them J1 VIDEO, J10 SDS-60J, J2 JOYSTICK, J3 >VALUE, J4 ., J5 RS232 + RETEA, J6 ., J7 FDD-CON, J8 FDD-CON, J9 .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

Commit message: Updated ICs values and positions
Parts:
- J3: value >VALUE -> MAB5SH
- UA8, UC8: value 2k x 4bit -> 2k x 4bit/-
- UB6: value ROM - 27C256 -> 27C256/27C512
- UE8A0: value 27128P -> 27128P/-

Commit message: Fix errors (IC & unnoticed cut for 1 EPROM)
Parts:
- added JX1: OPEN with 1 EPROM, HC2000:SolderJumper-2_P1.3mm_Open_Pad1.0x1.5mm, F.Cu at (480.1, 158.8)
- added JX2: CLOSED with 1 EPROM, HC2000:SolderJumper-2_P1.3mm_Open_Pad1.0x1.5mm, F.Cu at (508.0, 185.5)
- added JX3: CLOSED with 1 EPROM, HC2000:SolderJumper-2_P1.3mm_Open_Pad1.0x1.5mm, F.Cu at (501.5, 186.1)
- added JX4: CLOSED with 1 EPROM, HC2000:SolderJumper-2_P1.3mm_Open_Pad1.0x1.5mm, F.Cu at (478.3, 230.6)
- J3: value MAB5SH -> >VALUE
- SW1: value RESET_SW -> >VALUE
- UA1, UC7: value 74244N -> 74LS244
- UA11: value 7406N -> 74LS06
- UA23, UA34: value 7409N -> 74LS09
- UA8, UC8: value 2k x 4bit/- -> 2k x 4bit CMOS RAM/-
- UA9, UB10, UE4, UF8, UH10: value 74138N -> 74LS138
- UB1, UD10, UD3, UE10, UF10, UF4, UG12, UH12: value 7474N -> 74LS74
- UB12: value 74153N -> 74LS153
- UB2, UH3: value 7400N -> 74LS00
- UB3: value 74367N -> 74LS367
- UB9, UF7: value 74174N -> 74LS174
- UC1, UE11, UG0, UG4: value 7404N -> 74LS04
- UC10: value 74LS38N -> 74LS38
- UC12, UF3, UG3, UH1: value 74175N -> 74LS175
- UC2: value 7427N -> 74LS27
- UC3, UE3, UF9, UG9, UH8: value 7432N -> 74LS32
- UC4, UC5, UD5, UG7, UH6: value 74257N -> 74LS257
- UC6: value 74373N -> 74LS373
- UC9: value 74125N -> 74LS125
- UD1, UE2, UG11: value 7408N -> 74LS08
- UD11: value 7414N -> 74LS14
- UD12: value 74LS161N -> 74LS161
- UD4: value 74157N -> 74LS157
- UD6, UF6, UG6: value 74374N -> 74LS374
- UD7, UE7: value 41464 -> TMM41464AP-12
- UE6: value 74166N -> 74LS166
- UE8: value 8272 -> 8272 or D765AC-2
- UG1: value 7442N -> 74LS42
- UG10, UH5: value 7400N -> 74LS08
- UG8: value 7405N -> 74LS05
- UH11: value 7493N -> 74LS93
- UH4: value 7486N -> 74LS86
Connections:
- DX1 pad A: /HC2000_11/PHANTOM -> Net-(JX1-A)
- UA8 pad 8: Net-(UA8A-~{CS}) -> Net-(JX3-B)
- UB10 pad 14: Net-(UA8A-~{CS}) -> Net-(JX3-B)
- UC8 pad 8: Net-(UA8A-~{CS}) -> Net-(JX3-B)
- UD11 pad 12: /HC2000_11/PHANTOM -> Net-(JX2-B)
- UD11 pad 13: Net-(UA8A-~{CS}) -> Net-(JX3-A)
- UF10 pad 6: ROMFDD -> Net-(JX4-A)
- UX1 pad 18: Net-(UA8A-~{CS}) -> Net-(JX3-B)
Routing:
- net Net-(UA8A-~{CS}): track 235.3 -> 0.00 mm, vias 8 -> 0
- net Net-(JX1-A): track 0.00 -> 225.9 mm, vias 0 -> 4
- net Net-(JX3-B): track 0.00 -> 225.4 mm, vias 0 -> 8
- net /HC2000_11/PHANTOM: track 299.2 -> 107.6 mm, vias 7 -> 2
- net Net-(JX3-A): track 0.00 -> 7.16 mm
- net RDDATA: track 126.8 -> 121.7 mm
- net Net-(JX2-B): track 0.00 -> 4.68 mm
- net Net-(JX4-A): track 0.00 -> 4.55 mm
- net ROMFDD: track 369.8 -> 366.2 mm

Commit message: Revision-E
Parts:
- C14: value 100p/180p -> 180p
- C4: value 3,3uF/4,7uF -> 4,7uF
- C7: value 10p/15p -> 15p
- C8: value 220p/- -> -
- J3: value >VALUE -> MAB5SH
- R21: value 10k/470k -> 470k
- R22: value 8k2/6k -> 6k
- R26, R42, R45: value 330/- -> -
- R28, R40, R41, R56: value 220/1k -> 1k
- R30, R48: value 75/69 -> 69
- R31: value 240/270 -> 270
- R5, R60: value 330/300 -> 300
- R6: value 2M2/2M -> 2M
- R66: value 1k8/1k6 -> 1k6
- R68: value 5k6/5k1 -> 5k1
- SW1: value >VALUE -> RESET_SW
- T2: value 2N2369/2N2368 -> 2N2368
- T3: value 2N2369/BC108A -> BC108A
- UA8, UC8: value 2k x 4bit CMOS RAM/- -> -
- UB6: value 27C256/27C512 -> 27C512
- UE8A0: value 27128P/- -> -
Connections:
- JX2 pad 2: Net-(JX2-B) -> Net-(JX1-A)
- JX3 pad 2: Net-(JX3-B) -> Net-(JX3-A)
- JX4 pad 1: Net-(JX4-A) -> ROMFDD
- UA8 pad 8: Net-(JX3-B) -> Net-(JX3-A)
- UB10 pad 14: Net-(JX3-B) -> Net-(JX3-A)
- UC8 pad 8: Net-(JX3-B) -> Net-(JX3-A)
- UD11 pad 12: Net-(JX2-B) -> Net-(JX1-A)
- UF10 pad 6: Net-(JX4-A) -> ROMFDD
- UX1 pad 18: Net-(JX3-B) -> Net-(JX3-A)
Routing:
- net Net-(JX3-B): track 225.4 -> 0.00 mm, vias 8 -> 0
- net Net-(JX3-A): track 7.16 -> 232.5 mm, vias 0 -> 8
- net Net-(JX1-A): track 225.9 -> 230.6 mm
- net Net-(JX2-B): track 4.68 -> 0.00 mm
- net ROMFDD: track 366.2 -> 370.8 mm
- net Net-(JX4-A): track 4.55 -> 0.00 mm

Commit message: A few minor changes
R62 has value 470 instead of 910 and C6 is missing.
Connected a few conector's shield pins to GND.
Parts:
- C10: footprint HC2000:C025-025X050 -> HC2000:C025-024X044
- C11: footprint HC2000:C025-025X050 -> HC2000:C025-030X050
- C6: value 150p -> -
- R62: value 910 -> 470
- moved J10 0.25 mm to (399.7, 107.6)
- moved J3 0.25 mm to (365.3, 107.6)
- moved J4 0.25 mm to (399.7, 117.1)
Connections:
- J1 pad 0: (no net) -> GND
- J2 pad 0: (no net) -> GND
- J5 pad 0: (no net) -> GND
Routing:
- net GND: track 4393.3 -> 4429.5 mm, vias 25 -> 27
- net (no net): vias 14 -> 12
