File: HC2000.kicad_pcb (KiCad board)
At the start: 2 copper layers, 478 x 183 mm, 259 parts, among them J1 VIDEO, J10 SDS-60J, J2 JOYSTICK, J3 MAB5SH, J4 ., J5 RS232 + RETEA, J6 ., J7 FDD-CON, J8 FDD-CON, J9 .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

Commit message: Revision E final fixes before fork
Parts:
- added SilkFree: SilkFree, HC2000:SilkFree, F.Cu at (134.6, 139.8)
- L1: value 100 -> 100mH
Connections:
- UE10 pad 4: RESETL -> Net-(UD10A-PRE)
Routing:
- net RESETL: track 669.3 -> 658.8 mm
- net Net-(UD10A-PRE): track 53.4 -> 57.2 mm
Changed lines of the file:
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@@
       (net 1 "GND") (pinfunction "2") (pintype "passive"))
   )
+  (footprint "HC2000:SilkFree" (layer "F.Cu")
+    (at 134.645 139.775)
+    (attr smd)
+    (fp_text reference "SilkFree" (at 0 -0.5 unlocked) (layer "F.SilkS")
+        (effects (font (size 1 1) (thickness 0.15)))
+    )
+    (fp_text value "SilkFree" (at 0 1 unlocked) (layer "F.Fab")
+        (effects (font (size 1 1) (thickness 0.15)))
+    )
+    (pad "GND" smd oval (at 0 0) (size 10.16 78.74) (layers "F.Cu" "F.Paste")
+      (net 1 "GND") (thermal_bridge_angle 45))
+    (pad "GND" smd rect (at 0 0) (size 34.925 58.42) (layers "F.Cu" "F.Paste")
+      (net 1 "GND") (thermal_bridge_angle 45))
+    (group "" (id 7d01e9e2-c6a6-4964-80f0-52395fd1b52b)
+      (members
+        0b435667-cdd3-4339-bc29-5aa38792685d
+        2ad6b728-5013-4c89-a273-5ab9b7d9250e
+        40230df8-4d63-4842-a780-e89cd549daaf
+        912b1017-138f-4270-aacd-e84eedf8ca9c
+      )
+    )
+  )
   (footprint "HC2000:0204_7" (layer "F.Cu")
     (at 526.44 159.46 -90)
@@
       (net 280 "OUTF7") (pinfunction "CLK") (pintype "input"))
     (pad "4" thru_hole circle (at 0 3.81) (size 1.524 1.524) (drill 0.762) (layers "*.Cu" "*.Paste" "*.Mask")
-      (net 18 "RESETL") (pinfunction "PRE") (pintype "input"))
+      (net 85 "Net-(UD10A-PRE)") (pinfunction "PRE") (pintype "input"))
     (pad "5" thru_hole circle (at 2.54 3.81) (size 1.524 1.524) (drill 0.762) (layers "*.Cu" "*.Paste" "*.Mask")
       (net 425 "Net-(UE10A-Q)") (pinfunction "Q") (pintype "output"))
@@
         (effects (font (size 1.778 1.778) (thickness 0.1524)))
     )
-    (fp_text value "100" (at 3.81 6.35) (layer "F.SilkS") hide
+    (fp_text value "100mH" (at 3.81 6.35) (layer "F.SilkS") hide
         (effects (font (size 1.778 1.778) (thickness 0.1524)))
     )
@@
   (segment (start 311.81 123.9) (end 311.81 123.265) (width 0.3) (layer "B.Cu") (net 18))
   (segment (start 506.12 153.11) (end 506.12 156.285) (width 0.3) (layer "B.Cu") (net 18))
-  (segment (start 472.465 214.705) (end 471.83 215.34) (width 0.3) (layer "B.Cu") (net 18))
   (segment (start 313.08 121.995) (end 313.08 105.485) (width 0.3) (layer "B.Cu") (net 18))
   (segment (start 468.02 198.83) (end 468.02 196.29) (width 0.3) (layer "B.Cu") (net 18))
@@
   (segment (start 216.56 188.035) (end 216.56 183.59) (width 0.3) (layer "B.Cu") (net 18))
   (segment (start 470.56 226.77) (end 470.56 219.785) (width 0.3) (layer "B.Cu") (net 18))
-  (segment (start 471.83 218.515) (end 470.56 219.785) (width 0.3) (layer "B.Cu") (net 18))
   (segment (start 431.19 125.17) (end 431.19 158.19) (width 0.3) (layer "B.Cu") (net 18))
   (segment (start 468.02 234.39) (end 468.02 231.85) (width 0.3) (layer "B.Cu") (net 18))
@@
   (segment (start 562 127.71) (end 567.08 127.71) (width 0.3) (layer "B.Cu") (net 18))
   (segment (start 431.19 169.62) (end 431.19 164.54) (width 0.3) (layer "B.Cu") (net 18))
-  (segment (start 475.005 214.705) (end 472.465 214.705) (width 0.3) (layer "B.Cu") (net 18))
   (segment (start 211.48 234.39) (end 211.48 231.85) (width 0.3) (layer "B.Cu") (net 18))
   (segment (start 470.56 191.21) (end 470.56 189.94) (width 0.3) (layer "B.Cu") (net 18))
   (segment (start 211.48 234.39) (end 211.48 236.93) (width 0.3) (layer "B.Cu") (net 18))
   (segment (start 558.19 139.14) (end 558.19 131.52) (width 0.3) (layer "B.Cu") (net 18))
-  (segment (start 475.64 215.34) (end 475.005 214.705) (width 0.3) (layer "B.Cu") (net 18))
   (segment (start 217.83 182.32) (end 217.83 149.935) (width 0.3) (layer "B.Cu") (net 18))
   (segment (start 468.02 196.29) (end 470.56 193.75) (width 0.3) (layer "B.Cu") (net 18))
@@
   (segment (start 507.39 157.555) (end 507.39 170.89) (width 0.3) (layer "B.Cu") (net 18))
   (segment (start 470.56 229.31) (end 470.56 226.77) (width 0.3) (layer "B.Cu") (net 18))
-  (segment (start 471.83 215.34) (end 471.83 218.515) (width 0.3) (layer "B.Cu") (net 18))
   (segment (start 506.12 156.285) (end 507.39 157.555) (width 0.3) (layer "B.Cu") (net 18))
-  (segment (start 475.64 216.61) (end 475.64 215.34) (width 0.3) (layer "B.Cu") (net 18))
   (segment (start 431.19 158.19) (end 432.46 159.46) (width 0.3) (layer "B.Cu") (net 18))
   (segment (start 469.29 188.67) (end 469.29 170.255) (width 0.3) (layer "B.Cu") (net 18))
@@
   (via (at 470.56 205.18) (size 1.3335) (drill 0.762) (layers "F.Cu" "B.Cu") (net 85))
   (via (at 468.02 219.15) (size 1.3335) (drill 0.762) (layers "F.Cu" "B.Cu") (net 85))
+  (segment (start 475.64 216.61) (end 475.64 220.42) (width 0.3) (layer "B.Cu") (net 85))
   (segment (start 476.91 205.18) (end 476.91 219.15) (width 0.3) (layer "B.Cu") (net 85))
   (segment (start 475.64 198.83) (end 475.64 195.655) (width 0.3) (layer "B.Cu") (net 85))
@@
   (zone (net 1) (net_name "GND") (layer "F.Cu") (hatch none 0.1)
     (priority 6)
-    (connect_pads yes (clearance 0.508))
-    (min_thickness 0.025) (filled_areas_thickness no)
-    (fill yes (thermal_gap 0.025) (thermal_bridge_width 0.025))
-    (polygon
-      (pts
-        (xy 116.865 168.985)
-        (xy 116.865 110.565)
-        (xy 129.565 110.565)
-        (xy 129.565 104.215)
-        (xy 130.835 101.675)
-        (xy 134.01 100.405)
-        (xy 135.28 100.405)
-        (xy 138.455 101.675)
-        (xy 139.725 104.215)
-        (xy 139.725 110.565)
-        (xy 151.79 110.565)
-        (xy 151.79 168.985)
-        (xy 139.725 168.985)
-        (xy 139.725 175.335)
-        (xy 137.82 177.875)
-        (xy 135.28 179.145)
-        (xy 134.01 179.145)
-        (xy 131.47 177.875)
-        (xy 129.565 175.335)
-        (xy 129.565 168.985)
-      )
-    )
-  )
-  (zone (net 1) (net_name "GND") (layer "F.Cu") (hatch none 0.1)
-    (priority 6)

Commit message: Updated power, audio and keyboard connectors
Parts:
- added J11: Conn_02x10_Counter_Clockwise, HC2000:PinHeader_2x10_P2.54mm_Vertical, F.Cu at (197.5, 125.2)
- added J12: Ear_Jack, HC2000:Tayda_3.5mm_stereo_TRS_jack_A-853, F.Cu at (376.7, 106.0)
- added PS1: DD1718PA, HC2000:DD1718PA, F.Cu at (390.0, 117.9)
- J10: value SDS-60J -> Jack-DC; footprint HC2000:SDS-60J-CUI_SDS-60J -> HC2000:BarrelJack_Wuerth_6941xx301002
- J3: value MAB5SH -> Mic_Jack; footprint HC2000:MAB5SH -> HC2000:Tayda_3.5mm_stereo_TRS_jack_A-853
- J4: value . -> Jack-DC; footprint HC2000:HC-POWER -> HC2000:BarrelJack_Wuerth_6941xx301002
- moved J4 8.81 mm to (393.0, 111.3), turned to 180 degrees
- moved J10 7.32 mm to (406.0, 111.3)
- moved J3 3.06 mm to (362.7, 106.0), turned to 0 degrees
- moved JP2 1.80 mm to (384.8, 114.4), turned to 0 degrees
Connections:
- J10 pad 2: -12V -> GND
- J3 pad 1: MIC -> GND
- J3 pad 2: GND -> unconnected-(J3-Pad2)
- J3 pad 3: EAR -> unconnected-(J3-Pad3)
- J3 pad 4: unconnected-(J3-Pad4) -> MIC
- J3 pad 5: Net-(J3-Pad5) -> MIC
- J4 pad 3: -12V -> GND
- JP2 pad 2: Net-(J3-Pad5) -> unconnected-(JP2-Pad2)
- KB-CONN0 pad 10: unconnected-(KB-CONN0-Pad10) -> Net-(J11-Pin_13)
Routing:
- net MIC: track 205.6 -> 223.6 mm
- net BUSRQL: track 212.2 -> 230.1 mm, vias 5 -> 7
- net VCC: track 3906.0 -> 3890.3 mm
- net -12V: track 131.7 -> 118.9 mm
- net Net-(J3-Pad5): track 12.3 -> 0.00 mm
- net GND: track 4429.5 -> 4422.2 mm
- net Net-(SPEAKER0-2): track 84.0 -> 88.9 mm
- net +12V: track 175.9 -> 179.4 mm
- net EAR: track 12.2 -> 15.2 mm
- net TD3: track 86.3 -> 83.3 mm
- net TD1: track 92.1 -> 94.7 mm
- net TD4: track 64.4 -> 67.0 mm
- net TA11: track 69.5 -> 72.0 mm
- net Net-(J11-Pin_13): track 0.00 -> 2.54 mm
- net /HC2000_2/TA9: track 16.3 -> 18.8 mm
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