File: HC2000_4.kicad_sch (KiCad schematic)
At the start: 12 parts

Commit message: Fix errors (IC & unnoticed cut for 1 EPROM)
Parts:
- UB1, UF4: value 7474N -> 74LS74
- UB2: value 7400N -> 74LS00
- UC2: value 7427N -> 74LS27
- UC3, UE3: value 7432N -> 74LS32
- UD1: value 7408N -> 74LS08
- UH4: value 7486N -> 74LS86
Changed lines of the file:
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@@
       (effects (font (size 1.778 1.5113)) (justify left bottom))
     )
-    (property "Value" "7408N" (at 198.12 81.28 0)
+    (property "Value" "74LS08" (at 198.12 81.28 0)
       (effects (font (size 1.778 1.5113)) (justify left bottom))
     )
@@
       (effects (font (size 1.778 1.5113)) (justify left bottom))
     )
-    (property "Value" "7432N" (at 104.14 55.88 0)
+    (property "Value" "74LS32" (at 104.14 55.88 0)
       (effects (font (size 1.778 1.5113)) (justify left bottom))
     )
@@
       (effects (font (size 1.778 1.5113)) (justify left bottom))
     )
-    (property "Value" "7408N" (at 147.32 40.64 0)
+    (property "Value" "74LS08" (at 147.32 40.64 0)
       (effects (font (size 1.778 1.5113)) (justify left bottom))
     )
@@
       (effects (font (size 1.778 1.5113)) (justify left bottom))
     )
-    (property "Value" "7486N" (at 147.32 73.66 0)
+    (property "Value" "74LS86" (at 147.32 73.66 0)
       (effects (font (size 1.778 1.5113)) (justify left bottom))
     )
@@
       (effects (font (size 1.778 1.5113)) (justify left bottom))
     )
-    (property "Value" "7427N" (at 104.14 101.6 0)
+    (property "Value" "74LS27" (at 104.14 101.6 0)
       (effects (font (size 1.778 1.5113)) (justify left bottom))
     )
@@
       (effects (font (size 1.778 1.5113)) (justify left bottom))
     )
-    (property "Value" "7432N" (at 73.66 99.06 0)
+    (property "Value" "74LS32" (at 73.66 99.06 0)
       (effects (font (size 1.778 1.5113)) (justify left bottom))
     )
@@
       (effects (font (size 1.778 1.5113)) (justify left bottom))
     )
-    (property "Value" "7432N" (at 73.66 73.66 0)
+    (property "Value" "74LS32" (at 73.66 73.66 0)
       (effects (font (size 1.778 1.5113)) (justify left bottom))
     )
@@
       (effects (font (size 1.778 1.5113)) (justify left bottom))
     )
-    (property "Value" "7474N" (at 167.64 160.02 0)
+    (property "Value" "74LS74" (at 167.64 160.02 0)
       (effects (font (size 1.778 1.5113)) (justify left bottom))
     )
@@
       (effects (font (size 1.778 1.5113)) (justify left bottom))
     )
-    (property "Value" "7400N" (at 73.66 167.64 0)
+    (property "Value" "74LS00" (at 73.66 167.64 0)
       (effects (font (size 1.778 1.5113)) (justify left bottom))
     )
@@
       (effects (font (size 1.778 1.5113)) (justify left bottom))
     )
-    (property "Value" "7400N" (at 104.14 149.86 0)
+    (property "Value" "74LS00" (at 104.14 149.86 0)
       (effects (font (size 1.778 1.5113)) (justify left bottom))
     )
@@
       (effects (font (size 1.778 1.5113)) (justify left bottom))
     )
-    (property "Value" "7400N" (at 104.14 129.54 0)
+    (property "Value" "74LS00" (at 104.14 129.54 0)
       (effects (font (size 1.778 1.5113)) (justify left bottom))
     )
@@
       (effects (font (size 1.778 1.5113)) (justify left bottom))
     )
-    (property "Value" "7474N" (at 167.64 132.08 0)
+    (property "Value" "74LS74" (at 167.64 132.08 0)
       (effects (font (size 1.778 1.5113)) (justify left bottom))
     )
@@
       (effects (font (size 1.778 1.5113)) (justify left bottom))
     )
-    (property "Value" "7427N" (at 73.66 147.32 0)
+    (property "Value" "74LS27" (at 73.66 147.32 0)
       (effects (font (size 1.778 1.5113)) (justify left bottom))
     )
@@
       (effects (font (size 1.778 1.5113)) (justify left bottom))
     )
-    (property "Value" "7474N" (at 167.64 106.68 0)
-      (effects (font (size 1.778 1.5113)) (justify left bottom))
-    )
+    (property "Value" "74LS74" (at 167.64 106.68 0)
+      (effects (font (size 1.778 1.5113)) (justify left bottom))
+    )

Commit message: A few minor changes
R62 has value 470 instead of 910 and C6 is missing.
Connected a few conector's shield pins to GND.
Parts:
- C11: footprint HC2000:C025-025X050 -> HC2000:C025-030X050
Changed lines of the file:
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@@
       (effects (font (size 1.778 1.5113)) (justify left bottom))
     )
-    (property "Footprint" "HC2000:C025-025X050" (at 142.24 162.56 0)
+    (property "Footprint" "HC2000:C025-030X050" (at 142.24 162.56 0)
       (effects (font (size 1.27 1.27)) hide)
     )
