File: HC2000_12.kicad_sch (KiCad schematic)
At the start: 25 parts, among them T4 BC177, T5 BC177

Commit message: Fix errors (IC & unnoticed cut for 1 EPROM)
Parts:
- UC9: value 74125N -> 74LS125
- UD10, UE10: value 7474N -> 74LS74
- UE11: value 7404N -> 74LS04
- UF9: value 7432N -> 74LS32
Changed lines of the file:
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@@
       (effects (font (size 1.778 1.5113)) (justify left bottom))
     )
-    (property "Value" "7474N" (at 81.28 175.26 0)
+    (property "Value" "74LS74" (at 81.28 175.26 0)
       (effects (font (size 1.778 1.5113)) (justify left bottom))
     )
@@
       (effects (font (size 1.778 1.5113)) (justify left bottom))
     )
-    (property "Value" "74125N" (at 210.82 60.96 0)
+    (property "Value" "74LS125" (at 210.82 60.96 0)
       (effects (font (size 1.778 1.5113)) (justify left bottom))
     )
@@
       (effects (font (size 1.778 1.5113)) (justify left bottom))
     )
-    (property "Value" "7474N" (at 81.28 134.62 0)
+    (property "Value" "74LS74" (at 81.28 134.62 0)
       (effects (font (size 1.778 1.5113)) (justify left bottom))
     )
@@
       (effects (font (size 1.778 1.5113)) (justify left bottom))
     )
-    (property "Value" "7474N" (at 81.28 101.6 0)
+    (property "Value" "74LS74" (at 81.28 101.6 0)
       (effects (font (size 1.778 1.5113)) (justify left bottom))
     )
@@
       (effects (font (size 1.778 1.5113)) (justify left bottom))
     )
-    (property "Value" "7404N" (at 121.92 175.26 0)
+    (property "Value" "74LS04" (at 121.92 175.26 0)
       (effects (font (size 1.778 1.5113)) (justify left bottom))
     )
@@
       (effects (font (size 1.778 1.5113)) (justify left bottom))
     )
-    (property "Value" "7432N" (at 116.84 101.6 0)
+    (property "Value" "74LS32" (at 116.84 101.6 0)
       (effects (font (size 1.778 1.5113)) (justify left bottom))
     )
@@
       (effects (font (size 1.778 1.5113)) (justify left bottom))
     )
-    (property "Value" "7474N" (at 81.28 68.58 0)
+    (property "Value" "74LS74" (at 81.28 68.58 0)
       (effects (font (size 1.778 1.5113)) (justify left bottom))
     )
@@
       (effects (font (size 1.778 1.5113)) (justify left bottom))
     )
-    (property "Value" "74125N" (at 210.82 83.82 0)
+    (property "Value" "74LS125" (at 210.82 83.82 0)
       (effects (font (size 1.778 1.5113)) (justify left bottom))
     )
@@
       (effects (font (size 1.778 1.5113)) (justify left bottom))
     )
-    (property "Value" "74125N" (at 213.36 149.86 0)
-      (effects (font (size 1.778 1.5113)) (justify left bottom))
-    )
+    (property "Value" "74LS125" (at 213.36 149.86 0)
+      (effects (font (size 1.778 1.5113)) (justify left bottom))
+    )

Commit message: Revision-E
Parts:
- R22: value 8k2/6k -> 6k
Changed lines of the file:
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@@
       (effects (font (size 1.778 1.5113)) (justify left bottom))
     )
-    (property "Value" "8k2/6k" (at 201.422 115.57 0)
+    (property "Value" "6k" (at 201.422 115.57 0)
       (effects (font (size 1.778 1.5113)) (justify left bottom))
     )

Commit message: A few minor changes
R62 has value 470 instead of 910 and C6 is missing.
Connected a few conector's shield pins to GND.
Parts:
- UA10: Alt (none) -> 75188
- UF12: Alt (none) -> 75189
Changed lines of the file:
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@@
       (effects (font (size 1.27 1.27)) hide)
+    )
+    (property "Alt" "75188" (at 119.38 68.58 0)
+      (effects (font (size 1.27 1.27)))
     )
     (pin "1")
@@
       (effects (font (size 1.27 1.27)) hide)
     )
-    (pin "1")
+    (property "Alt" "75189" (at 177.8 55.88 0)
+      (effects (font (size 1.27 1.27)))
+    )
+    (pin "1")

Commit message: Revision E final fixes before fork
Connections:
- net RESETL: no longer UE10.4 (PRE)
- net at R44.1, UD10.10 (PRE), UD10.4 (PRE)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: now also UE10.4 (PRE)
Changed lines of the file:
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@@
   (junction (at 154.94 104.14) (diameter 0) (color 0 0 0 0)
   )
+  (junction (at 68.58 119.38) (diameter 0) (color 0 0 0 0)
+  )
   (junction (at 198.12 134.62) (diameter 0) (color 0 0 0 0)
   )
@@
   (junction (at 71.12 96.52) (diameter 0) (color 0 0 0 0)
   )
-  (junction (at 71.12 119.38) (diameter 0) (color 0 0 0 0)
-  )
   (junction (at 177.8 104.14) (diameter 0) (color 0 0 0 0)
   )
@@
     (stroke (width 0) (type default))
   )
-  (wire (pts (xy 71.12 119.38) (xy 76.2 119.38))
-    (stroke (width 0) (type default))
-  )
   (wire (pts (xy 210.82 132.08) (xy 210.82 134.62))
     (stroke (width 0) (type default))
@@
     (stroke (width 0) (type default))
   )
-  (wire (pts (xy 71.12 119.38) (xy 71.12 139.7))
-    (stroke (width 0) (type default))
-  )
   (wire (pts (xy 165.1 40.64) (xy 165.1 48.26))
     (stroke (width 0) (type default))
@@
     (stroke (width 0) (type default))
   )
+  (wire (pts (xy 68.58 119.38) (xy 76.2 119.38))
+    (stroke (width 0) (type default))
+  )
   (wire (pts (xy 147.32 104.14) (xy 147.32 114.3))
     (stroke (width 0) (type default))
@@
     (stroke (width 0) (type default))
   )
+  (wire (pts (xy 68.58 119.38) (xy 68.58 129.54))
+    (stroke (width 0) (type default))
+  )
   (wire (pts (xy 76.2 63.5) (xy 71.12 63.5))
     (stroke (width 0) (type default))
@@
     (stroke (width 0) (type default))
   )
-  (wire (pts (xy 68.58 86.36) (xy 68.58 129.54))
+  (wire (pts (xy 68.58 86.36) (xy 68.58 119.38))
     (stroke (width 0) (type default))
   )
@@
     (stroke (width 0) (type default))
   )
-  (wire (pts (xy 71.12 96.52) (xy 71.12 119.38))
-    (stroke (width 0) (type default))
-  )
+  (wire (pts (xy 71.12 96.52) (xy 71.12 139.7))
+    (stroke (width 0) (type default))
+  )
